File: hardware/pcb/NES_II/NES_II.kicad_pcb (KiCad board)
At the start: 2 copper layers, 110 x 100 mm, 25 parts, among them J1 Conn_01x02, J2 Conn_01x02, J3 Conn_01x03, U1 GAL16V8, U2 74HC244

Commit message: PCB revision 2
Parts:
- removed J1, J2: Conn_01x02, Connector_PinHeader_2.54mm:PinHeader_1x02_P2.54mm_Vertical
- removed J3: Conn_01x03, Connector_PinHeader_2.54mm:PinHeader_1x03_P2.54mm_Vertical
- removed PI1: Conn_01x11_Male, Connector_PinSocket_2.54mm:PinSocket_1x11_P2.54mm_Vertical
- removed R1: R, Resistor_THT:R_Axial_DIN0207_L6.3mm_D2.5mm_P10.16mm_Horizontal
- removed U2: 74HC244, Package_DIP:DIP-20_W7.62mm_LongPads
- added C6: 10uf, Capacitor_THT:C_Disc_D3.8mm_W2.6mm_P2.50mm, F.Cu at (91.9, 102.4)
- added C7: C, Capacitor_THT:CP_Radial_Tantal_D4.5mm_P2.50mm, F.Cu at (97.3, 102.3)
- added R2: 10k, Resistor_THT:R_Axial_DIN0204_L3.6mm_D1.6mm_P5.08mm_Vertical, F.Cu at (86.6, 101.1)
- added R3: 1k, Resistor_THT:R_Axial_DIN0204_L3.6mm_D1.6mm_P5.08mm_Horizontal, F.Cu at (69.1, 95.8)
- added U3: 74HC74, Package_DIP:DIP-14_W7.62mm, F.Cu at (91.9, 111.5)
- C4: value C -> 33pf
- moved C4 70.0 mm to (79.8, 97.5), turned to 90 degrees
- moved C3 43.2 mm to (41.9, 96.3)
- moved C2 26.7 mm to (97.0, 131.1), turned to 0 degrees
- moved C1 20.8 mm to (71.4, 100.8), turned to 0 degrees
- moved U1 19.4 mm to (79.2, 128.0)
- moved PRG_RAM1 17.6 mm to (50.5, 98.6)
- moved BIOS_ROM1 15.7 mm to (25.7, 100.6)
- moved NEG5_IN1 10.9 mm to (66.0, 185.5)
- moved AII_MEZZ1 6.43 mm to (27.9, 175.0)
- moved NEG12_IN1 6.41 mm to (71.1, 185.6)
- moved 12V_IN1 5.72 mm to (54.8, 185.7)
- moved GND1 3.35 mm to (60.5, 185.7)
- moved CHAR_RAM1 0.11 mm to (92.7, 152.4)
Connections:
- AII_MEZZ1 pad 1: AII_IOSELB -> +5V
- AII_MEZZ1 pad 11: /CA4 -> GND
- AII_MEZZ1 pad 13: /CA5 -> +5V
- AII_MEZZ1 pad 15: /CA6 -> +5V
- AII_MEZZ1 pad 17: /CA7 -> +5V
- AII_MEZZ1 pad 19: /CA8 -> GND
- AII_MEZZ1 pad 21: /CA9 -> GND
- AII_MEZZ1 pad 23: /CA10 -> GND
- AII_MEZZ1 pad 25: /CA11 -> GND
- AII_MEZZ1 pad 27: /CA12 -> GND
- AII_MEZZ1 pad 28: AII_Q3 -> M2
- AII_MEZZ1 pad 29: /CA13 -> GND
- AII_MEZZ1 pad 31: /CA14 -> +5V
- AII_MEZZ1 pad 39: AII_IOSTROBEB -> +5V
- AII_MEZZ1 pad 40: AII_RESB -> SW_RST
- BIOS_ROM1 pad 1: /CA14 -> +5V
- CHAR_RAM1 pad 2: /PA12 -> /PA6
- CHAR_RAM1 pad 23: /PA11 -> /PA2
- CHAR_RAM1 pad 4: /PA6 -> /PA5
- CHAR_RAM1 pad 5: /PA5 -> /PA4
- CHAR_RAM1 pad 6: /PA4 -> /PA3
- CHAR_RAM1 pad 7: /PA3 -> /PA11
- CHAR_RAM1 pad 8: /PA2 -> /PA12
- PRG_RAM1 pad 1: /CA14 -> RAM_A14
- PRG_RAM1 pad 26: /CA13 -> RAM_A13
- U1 pad 12: AII_IOSELB -> RAM_A13
- U1 pad 14: AII_IOSTROBEB -> CIRAM_A10
- U1 pad 15: DBG_RDB -> SW_CLK
- U1 pad 16: DBG_WRB -> RAM_A14
- U1 pad 2: /CA8 -> SWA
- U1 pad 3: /CA9 -> SWB
- U1 pad 4: /CA10 -> /PA10
- U1 pad 5: /CA11 -> /PA11
- U1 pad 9: M2 -> Net-(C4-Pad1)
Routing:
- net CIRAM_A10: track 9.46 -> 387.9 mm
- net SW_RST: track 0.00 -> 253.8 mm
- net /PA11: track 75.0 -> 323.7 mm
- net /PA10: track 65.4 -> 303.9 mm
- net /CA11: track 351.9 -> 138.3 mm
- net AII_IOSELB: track 201.1 -> 0.00 mm, vias 1 -> 0
- net /CA14: track 275.0 -> 89.9 mm
- net DBG_WRB: track 135.3 -> 0.00 mm, vias 1 -> 0
- net /CA7: track 286.7 -> 153.1 mm
- net /CA8: track 279.4 -> 146.2 mm
- net /CA6: track 279.2 -> 149.8 mm
- net DBG_RDB: track 128.5 -> 0.00 mm
- net /CA13: track 278.8 -> 151.2 mm
- net /CA9: track 270.4 -> 143.8 mm
- net ROMSELB: track 78.2 -> 204.2 mm, vias 1 -> 0
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Other:
- outline, holes or cut-outs redrawn
