File: hardware/pcb/NES_II/NES_II.kicad_sch (KiCad schematic)
At the start: 21 parts, among them J1 Conn_01x02, J2 Conn_01x02, J3 Conn_01x03, U1 GAL16V8, U2 74HC244

Commit message: PCB revision 2
Parts:
- removed J1, J2: Conn_01x02, Connector_PinHeader_2.54mm:PinHeader_1x02_P2.54mm_Vertical, symbol Connector_Generic:Conn_01x02
- removed J3: Conn_01x03, Connector_PinHeader_2.54mm:PinHeader_1x03_P2.54mm_Vertical, symbol Connector_Generic:Conn_01x03
- removed PI1: Conn_01x11_Male, Connector_PinSocket_2.54mm:PinSocket_1x11_P2.54mm_Vertical, symbol Connector:Conn_01x11_Male
- removed R1: R, Resistor_THT:R_Axial_DIN0207_L6.3mm_D2.5mm_P15.24mm_Horizontal, symbol Device:R
- removed U2: 74HC244, Package_DIP:DIP-20_W7.62mm_LongPads, symbol 74xx:74HC244
- added C6: 10uf, Capacitor_THT:C_Disc_D3.8mm_W2.6mm_P2.50mm, symbol Device:C
- added C7: C, Capacitor_THT:CP_Radial_Tantal_D4.5mm_P2.50mm, symbol Device:C
- added R2: 10k, Resistor_THT:R_Axial_DIN0204_L3.6mm_D1.6mm_P5.08mm_Vertical, symbol Device:R
- added R3: 1k, Resistor_THT:R_Axial_DIN0204_L3.6mm_D1.6mm_P5.08mm_Horizontal, symbol Device:R
- added U3: 74HC74, Package_DIP:DIP-14_W7.62mm, symbol 74xx:74HC74
- C4: value C -> 33pf
Connections:
- net AII_Q3 is gone; now on net M2: AII_MEZZ1.28 (Pin_28)
- net +5V: now also AII_MEZZ1.1 (Pin_1), AII_MEZZ1.13 (Pin_13), AII_MEZZ1.15 (Pin_15), AII_MEZZ1.17 (Pin_17), AII_MEZZ1.31 (Pin_31), AII_MEZZ1.39 (Pin_39), BIOS_ROM1.1 (A14), C7.1, R2.1, U3.10 (~{S}), U3.14 (VCC), U3.4 (~{S})
- net CA10: no longer AII_MEZZ1.23 (Pin_23), U1.4 (I4)
- net CA11: no longer AII_MEZZ1.25 (Pin_25), U1.5 (I5)
- net CA12: no longer AII_MEZZ1.27 (Pin_27)
- net CA13: no longer AII_MEZZ1.29 (Pin_29), PRG_RAM1.26 (A13)
- net CA14: no longer AII_MEZZ1.31 (Pin_31), BIOS_ROM1.1 (A14), PRG_RAM1.1 (A14)
- net CA4: no longer AII_MEZZ1.11 (Pin_11)
- net CA5: no longer AII_MEZZ1.13 (Pin_13)
- net CA6: no longer AII_MEZZ1.15 (Pin_15)
- net CA7: no longer AII_MEZZ1.17 (Pin_17)
- net CA8: no longer AII_MEZZ1.19 (Pin_19), U1.2 (I2)
- net CA9: no longer AII_MEZZ1.21 (Pin_21), U1.3 (I3)
- net CD0: now also U3.12 (D)
- net CD1: now also U3.2 (D)
- net CIRAM_A10: now also U1.14 (IO6)
- net GND: now also AII_MEZZ1.11 (Pin_11), AII_MEZZ1.19 (Pin_19), AII_MEZZ1.21 (Pin_21), AII_MEZZ1.23 (Pin_23), AII_MEZZ1.25 (Pin_25), AII_MEZZ1.27 (Pin_27), AII_MEZZ1.29 (Pin_29), C6.2, C7.2, U3.7 (GND)
- net M2: now also R3.1; no longer U1.9 (I9)
- net PA10: now also U1.4 (I4)
- net PA11: now also CHAR_RAM1.7 (A3), U1.5 (I5); no longer CHAR_RAM1.23 (A11)
- net PA12: now also CHAR_RAM1.8 (A2); no longer CHAR_RAM1.2 (A12)
- net PA2: now also CHAR_RAM1.23 (A11); no longer CHAR_RAM1.8 (A2)
- net PA3: now also CHAR_RAM1.6 (A4); no longer CHAR_RAM1.7 (A3)
- net PA4: now also CHAR_RAM1.5 (A5); no longer CHAR_RAM1.6 (A4)
- net PA5: now also CHAR_RAM1.4 (A6); no longer CHAR_RAM1.5 (A5)
- net PA6: now also CHAR_RAM1.2 (A12); no longer CHAR_RAM1.4 (A6)
- net at C4.1: now also U1.9 (I9), R3.2
- net AII_IOSELB renamed RAM_A13
- net RAM_A13: now also PRG_RAM1.26 (A13); no longer AII_MEZZ1.1 (Pin_1)
- removed net AII_IOSTROBEB: AII_MEZZ1.39 (Pin_39), U1.14 (IO6)
- net AII_RESB renamed SW_RST
- net SW_RST: now also C6.1, R2.2, U3.1 (~{R}), U3.13 (~{R})
- net DBG_RDB renamed SW_CLK
- net SW_CLK: now also U3.11 (C), U3.3 (C)
- net DBG_WRB renamed RAM_A14
- net RAM_A14: now also PRG_RAM1.1 (A14)
- new net SWA: U1.2 (I2), U3.9 (Q)
- new net SWB: U1.3 (I3), U3.5 (Q)
Other:
- moved on the sheet: AII_MEZZ1, BIOS_ROM1, C1, C2, C3, C5, PRG_RAM1, U1
